File: pcb/TK44/TK44.kicad_pcb (KiCad board)
At the start: 2 copper layers, 289.9 x 99.6 mm, 117 parts, among them J1 BATT, J2 SWD, J3 USB_C_Receptacle_USB2.0, Q1 AO3407, SW1 MX, SW10 MX, SW11 MX, SW12 MX, SW13 MX, SW14 MX, SW15 MX, SW16 MX, SW17 MX, SW18 MX, SW19 MX, SW2 MX, SW20 MX, SW21 MX, SW22 MX, SW23 MX, SW24 MX, SW25 MX, SW26 MX, SW27 MX, SW28 MX, SW29 MX, SW3 MX, SW30 MX, SW31 MX, SW32 MX, SW33 MX, SW34 MX, SW35 MX, SW36 MX, SW37 MX, SW38 MX, SW39 MX, SW4 MX, SW40 MX, SW41 MX, SW42 MX, SW43 MX, SW44 MX, SW45 SW_DPDT, SW5 MX, SW6 MX, SW7 MX, SW8 MX, SW9 MX, U1 HOLYIOT-18010, U2 MCP73831, U3 XC6220-3.3V

Commit message: Fix DRC errors and silk overlapping
Parts:
- R1: value 5.1K -> R1
- R2: value 5.1K -> R2
- R3: value 1K -> R3
- R4: value 810K -> R4
- R5: value 1K -> R5
- R6: value 3.3K -> R6
- R7: value 2M -> R7
- R8: value 100K -> R8
Routing:
- net /P0.30: track 135.5 -> 146.3 mm
- net /P0.31: track 122.7 -> 132.8 mm
- net /P0.04: track 139.1 -> 146.2 mm
- net /P0.28: track 86.6 -> 89.8 mm
- net /P0.29: track 113.7 -> 116.2 mm
- net /P1.00: track 127.6 -> 128.8 mm
- net /P1.03: track 108.9 -> 109.8 mm
