File: pcb/TK44/TK44.kicad_sch (KiCad schematic)
At the start: 108 parts, among them J1 BATT, J2 SWD, J3 USB_C_Receptacle_USB2.0, Q1 AO3407, SW1 MX, SW10 MX, SW11 MX, SW12 MX, SW13 MX, SW14 MX, SW15 MX, SW16 MX, SW17 MX, SW18 MX, SW19 MX, SW2 MX, SW20 MX, SW21 MX, SW22 MX, SW23 MX, SW24 MX, SW25 MX, SW26 MX, SW27 MX, SW28 MX, SW29 MX, SW3 MX, SW30 MX, SW31 MX, SW32 MX, SW33 MX, SW34 MX, SW35 MX, SW36 MX, SW37 MX, SW38 MX, SW39 MX, SW4 MX, SW40 MX, SW41 MX, SW42 MX, SW43 MX, SW44 MX, SW45 SW_DPDT, SW5 MX, SW6 MX, SW7 MX, SW8 MX, SW9 MX, U1 HOLYIOT-18010, U2 TP4054, U3 AP2112K-3.3

Commit message: No comment /////
Parts:
- D1, D10, D11, D12, D13, D14, D15, D16, D17, D18, D19, D2, D20, D21, D22, D23, D24, D25, D26, D27, D28, D29, D3, D30, D31, D32, D33, D34, D35, D36, D37, D38, D39, D4, D40, D41, D42, D43, D44, D46, D5, D6, D7, D8, D9: footprint space-invader:D_SOD-123 -> TK44:D_SOD-123
- D45, D47: footprint (none) -> TK44:LED_0603
- J1: footprint space-invader:Battery_Holder_18650_Nickel -> TK44:Battery_Connector
- J2: footprint space-invader:Connector_THT_1x4_2.54 -> TK44:Connector_THT_1x4_2.54
- J3: footprint space-invader:USB-C-PCB -> TK44:USB-C-C168688
- Q1: footprint space-invader:SOT-23 -> TK44:SOT-23
- R1, R2, R4, R7, R8: footprint space-invader:R_0603 -> TK44:R_0603
- R3, R5: footprint (none) -> TK44:R_0603
- R6: value R_Small -> 3.3K; footprint (none) -> TK44:R_0603
- SW1, SW10, SW11, SW12, SW13, SW14, SW15, SW16, SW17, SW18, SW19, SW2, SW20, SW21, SW22, SW23, SW24, SW25, SW26, SW27, SW28, SW29, SW3, SW30, SW31, SW32, SW33, SW34, SW35, SW36, SW39, SW4, SW42, SW5, SW6, SW7, SW8, SW9: footprint space-invader:Switch_Mx_Hotswap_1u -> TK44:Switch_Mx_Hotswap_1u
- SW37, SW44: footprint space-invader:Switch_Mx_Hotswap_1.5u -> TK44:Switch_Mx_Hotswap_1u
- SW38, SW40, SW41, SW43: footprint space-invader:Switch_Mx_Hotswap_1u -> TK44:Switch_Mx_Hotswap_1.25u
- SW45: footprint space-invader:MSK-12C02 -> TK44:MSK-12C02
- SWT1: footprint space-invader:K2-1187SQ -> TK44:K2-1187SQ
- U1: footprint space-invader:Holyiot-18010-nRF52840 -> TK44:Holyiot-18010-nRF52840
- U2: value TP4054 -> MCP73831; footprint Package_TO_SOT_SMD:SOT-23-5 -> TK44:SOT-23-5
- U3: value AP2112K-3.3 -> XC6220-3.3V; footprint space-invader:SOT-23-5 -> TK44:SOT-23-5
Connections:
- net VBUT is gone; now on net VBAT: U2.3 (VBAT)
- net P0.04: now also SW11.2, SW23.2, SW35.2; no longer SW14.2, SW2.2, SW26.2
- net P0.05: now also SW12.2, SW24.2, SW36.2, SW44.2; no longer SW1.2, SW13.2, SW25.2, SW37.2
- net P0.12: no longer SW12.2, SW24.2, SW36.2, SW44.2
- net P0.22: now also SW1.2, SW13.2, SW25.2, SW37.2; no longer SW11.2, SW23.2, SW35.2
- net P0.28: now also SW19.2, SW31.2, SW41.2, SW7.2; no longer SW18.2, SW30.2, SW40.2, SW6.2
- net P0.29: now also SW20.2, SW32.2, SW42.2, SW8.2; no longer SW17.2, SW29.2, SW39.2, SW5.2
- net P0.30: now also SW21.2, SW33.2, SW43.2, SW9.2; no longer SW16.2, SW28.2, SW38.2, SW4.2
- net P0.31: now also SW10.2, SW22.2, SW34.2; no longer SW15.2, SW27.2, SW3.2
- net P1.00: now also SW14.2, SW2.2, SW26.2; no longer SW10.2, SW22.2, SW34.2
- net P1.01: now also SW16.2, SW28.2, SW38.2, SW4.2; no longer SW20.2, SW32.2, SW42.2, SW8.2
- net P1.02: now also SW17.2, SW29.2, SW39.2, SW5.2; no longer SW19.2, SW31.2, SW41.2, SW7.2
- net P1.03: now also SW15.2, SW27.2, SW3.2; no longer SW21.2, SW33.2, SW43.2, SW9.2
- net P1.04: now reaches U1.33 (P1.04)
- net P1.04: now also SW18.2, SW30.2, SW40.2, SW6.2
- net P0.03: no longer names the net of U1.6 (P0.03/AIN1)

Commit message: Change battery pin
Connections:
- net BT_PIN: now reaches U1.7 (P0.02/AIN0)
- net BT_PIN: now also R4.2, R7.1
- removed net BATTERY_PIN: R4.2, R7.1, U1.20 (P0.19)
Changed lines of the file:
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@@
   (no_connect (at 58.42 160.655))
   (no_connect (at 37.465 71.755))
-  (no_connect (at 23.495 43.815))
   (no_connect (at 47.625 71.755))
   (no_connect (at 23.495 41.275))
+  (no_connect (at 50.165 71.755))
   (no_connect (at 19.05 139.065))
   (no_connect (at 41.91 131.445))
@@
     (stroke (width 0) (type solid) (color 0 0 0 0))
   )
+  (wire (pts (xy 20.955 43.815) (xy 23.495 43.815))
+    (stroke (width 0) (type default) (color 0 0 0 0))
+  )
   (wire (pts (xy 187.325 68.58) (xy 201.295 68.58))
     (stroke (width 0) (type default) (color 0 0 0 0))
@@
     (stroke (width 0) (type default) (color 0 0 0 0))
   )
-  (wire (pts (xy 50.165 71.755) (xy 50.165 74.295))
-    (stroke (width 0) (type default) (color 0 0 0 0))
-  )
   (wire (pts (xy 41.91 121.285) (xy 46.99 121.285))
     (stroke (width 0) (type solid) (color 0 0 0 0))
@@
     (effects (font (size 1.27 1.27)) (justify right bottom))
   )
-  (label "BATTERY_PIN" (at 50.165 74.295 270)
+  (label "BT_PIN" (at 20.955 43.815 180)
     (effects (font (size 1.27 1.27)) (justify right bottom))
   )
@@
     (effects (font (size 1.27 1.27)) (justify right bottom))
   )
-  (label "BATTERY_PIN" (at 27.94 179.705 180)
-    (effects (font (size 1.27 1.27)) (justify right bottom))
-  )
+  (label "BT_PIN" (at 27.94 179.705 180)
+    (effects (font (size 1.27 1.27)) (justify right bottom))
+  )
